File: PCBs/ButtonMountingBoard2x3Way/ButtonMountingBoard2x3Way.kicad_sch (KiCad schematic)
At the start: 34 parts, among them J1 Conn_01x06_Male, J2 Conn_01x10_Male, J3 Conn_01x06_Male, SW1 SW_TACT_LED, SW2 SW_TACT_LED, SW3 SW_TACT_LED, SW4 SW_TACT_LED, SW5 SW_TACT_LED, SW6 SW_TACT_LED, SW7 SW_TACT_LED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

Commit message: V1.1 PCB updates after initial testing 1. Share data out line between LCD, 7 Segment and button scan to yield spare io lines for    control of WS8212 LEDs for music stand lamp 2. Replace level shifting FET on Button Driver PCBs by resistor 3. Generate combined ks61,button driver & button mount prototype PCB for economic testing with JLC PCB
Parts:
- removed D4, D5: 1N4148, Diode_SMD:D_SOD-123, symbol Device:D
- removed H4: MountingHole, MountingHole:MountingHole_2.7mm_M2.5, symbol Mechanical:MountingHole
- removed J1, J3: Conn_01x06_Male, Connector_PinHeader_2.54mm:PinHeader_1x06_P2.54mm_Vertical, symbol Connector:Conn_01x06_Male
- removed J2: Conn_01x10_Male, Connector_PinHeader_2.54mm:PinHeader_1x10_P2.54mm_Vertical, symbol Connector:Conn_01x10_Male
- removed R4, R5: 560, Resistor_SMD:R_0805_2012Metric_Pad1.20x1.40mm_HandSolder, symbol Device:R
- removed SW4, SW5: SW_TACT_LED, New_Library_fp:TS12_TS27, symbol New_Library:SW_TACT_LED
- added JB1, JB2, JB3, JB4: Conn_01x05_Male, Connector_PinHeader_2.54mm:PinHeader_1x05_P2.54mm_Vertical, symbol Connector:Conn_01x05_Male
Connections:
- net SW8: now reaches D8.2 (A), R8.2
- net SW8: now also JB3.3 (Pin_3), JB4.3 (Pin_3)
- net SW6: now reaches D6.2 (A), R6.2
- net SW6: now also JB3.1 (Pin_1), JB4.1 (Pin_1)
- net SW1: now reaches D1.2 (A), R1.2
- net SW1: now also JB1.1 (Pin_1), JB2.1 (Pin_1)
- net SW2: now reaches D2.2 (A), R2.2
- net SW2: now also JB1.2 (Pin_2), JB2.2 (Pin_2)
- net SW3: now reaches D3.2 (A), R3.2
- net SW3: now also JB1.3 (Pin_3), JB2.3 (Pin_3)
- net SW7: now reaches D7.2 (A), R7.2
- net SW7: now also JB3.2 (Pin_2), JB4.2 (Pin_2)
- net LED renamed 0V
- net 0V: now also JB1.4 (Pin_4), JB2.4 (Pin_4); no longer SW6.5, SW7.5, SW8.5
- net SW renamed SW1-3
- net SW1-3: now also JB1.5 (Pin_5), JB2.5 (Pin_5); no longer SW6.3, SW6.4, SW7.3, SW7.4, SW8.3, SW8.4
- new net 0v: JB3.4 (Pin_4), JB4.4 (Pin_4), SW6.5, SW7.5, SW8.5
- new net SW6-8: JB3.5 (Pin_5), JB4.5 (Pin_5), SW6.3, SW6.4, SW7.3, SW7.4, SW8.3, SW8.4
Other:
- note added: "SW1 SW2 SW3 0V SW"
- note added: "SW6 SW7 SW8 0V SW"
- note added: "V1.0 Initial Release"
- note removed: "V1.0 Initial Release V1.1 R1-R8 270R->560R, Trim PCB bottom 1mm, 180 Rot R1, Silk screen fixes"
