File: PCBs/MidiInterfaceKS61/MidiInterfaceKS61.kicad_pcb (KiCad board)
At the start: 2 copper layers, 68.6 x 45.7 mm, 82 parts, among them CN13 Conn_01x13_Male, CN14 Conn_01x12_Male, J3 Conn_01x20_Female, J4 Conn_01x20_Female, J5 Conn_01x01_Male

Commit message: V1.1 PCB updates after initial testing 1. Share data out line between LCD, 7 Segment and button scan to yield spare io lines for    control of WS8212 LEDs for music stand lamp 2. Replace level shifting FET on Button Driver PCBs by resistor 3. Generate combined ks61,button driver & button mount prototype PCB for economic testing with JLC PCB
Parts:
- added J6: LAMP, Connector_PinHeader_2.54mm:PinHeader_2x03_P2.54mm_Vertical, F.Cu at (151.1, 114.3)
- added POT1: Conn_01x02_Male, Connector_PinHeader_2.54mm:PinHeader_1x02_P2.54mm_Vertical, F.Cu at (190.5, 81.3)
- RD32: value 4k7 -> 3K3
- RU14, RU15: value *4k7 -> 4k7
- RU32: value 4k7* -> 4k7
- moved RU33 16.7 mm to (196.8, 97.8), turned to 0 degrees
- moved RU34 14.7 mm to (196.8, 95.2), turned to 0 degrees
- moved J5 2.55 mm to (139.7, 116.8)
Connections:
- net /GND renamed /0V
- Buttons1 pad 3: /PB10 -> /PB7
- SEG7 pad 3: /PA13 -> /PB7
- SEG7 pad 4: /PA14 -> /PB10
Routing:
- net /PB7: track 31.4 -> 152.2 mm
- net /PA14: track 29.5 -> 75.7 mm, vias 0 -> 1
- net /PA13: track 31.1 -> 74.3 mm
- net /PB10: track 22.5 -> 57.5 mm
- net /0V: track 250.8 -> 283.9 mm, vias 0 -> 6
- net /3V3: track 50.2 -> 73.9 mm
- net /PC13: track 18.3 -> 20.8 mm
- net /PB13: track 29.3 -> 31.3 mm
- net /PB6: track 30.6 -> 32.6 mm
- net /PB9: track 16.4 -> 18.3 mm
- net /5V: track 221.4 -> 220.6 mm
Other:
- board text added: "'SCOPE"
- board text added: "0V 3V3"
- board text added: "0V 5V PB7B11B12"
- board text added: "0V A13 5V"
- board text added: "0V A14 5V"
- board text added: "0V PULLDOWN"
- board text added: "3V3 0V"
- board text added: "5V 0V PB7B10C13"
- board text added: "5V A13 0V"
- board text added: "5V A14 0V"
- board text added: "5V PULLUP"
- board text added: "A13 A14"
- board text added: "B12B11PB7 5V 0V"
- board text added: "C13B10PB7 0V 5V"
- board text added: "FIT3k3"
- board text added: "KS61 MIDI INTERFACE V1.1"
- board text added: "LAMP"
- board text removed: "* *"
- board text removed: "0V 5V B12B11B10"
- board text removed: "5V 0V A13A14C13"
- board text removed: "B12B11B10 5V 0V"
- board text removed: "C13A14A13 0V 5V"
- board text removed: "KS61 MIDI INTERFACE V1.0"
- board text removed: "PULLDOWN"
- board text removed: "PULLUP"
