File: PCBs/WiredButtonDriver/WiredButtonDriver.kicad_pcb (KiCad board)
At the start: 2 copper layers, 78.7 x 22.9 mm, 35 parts, among them J6 IN, J7 OUT, Q1 AO3400A, U2 74HC164

Commit message: V1.1 PCB updates after initial testing 1. Share data out line between LCD, 7 Segment and button scan to yield spare io lines for    control of WS8212 LEDs for music stand lamp 2. Replace level shifting FET on Button Driver PCBs by resistor 3. Generate combined ks61,button driver & button mount prototype PCB for economic testing with JLC PCB
Parts:
- removed Q1: AO3400A, Package_TO_SOT_SMD:SOT-23
- removed R9: 10k, Resistor_SMD:R_0805_2012Metric_Pad1.20x1.40mm_HandSolder
- R10: value 270 -> 1K
- R11, R12, R13, R14, R15, R16, R17, R18: value 270 -> 560
Connections:
- R10 pad 1: Net-(Q1-Pad1) -> Net-(J6-Pad5)
Routing:
- net /0V: track 153.5 -> 131.5 mm
- net Net-(Q1-Pad1): track 9.64 -> 0.00 mm
- net Net-(J6-Pad5): track 99.9 -> 107.4 mm
Other:
- board text added: "0V 5V DINCLKBUT"
- board text added: "0V 5V DIPCLKBUT"
- board text added: "0V 5V DOPCLKBUT"
- board text added: "1"
- board text added: "Wired Button+LED Driver V1.1"
- board text removed: "AO3400"
- board text removed: "Wired Button+LED Driver V1.0"
